File: KiCad/PC8001-PSG.kicad_sch (KiCad schematic)
At the start: 26 parts, among them J1 AudioJack, J2 PC-8001 Ext BUS, U1 74LS32, U2 74LS74, U3 74LS138, U4 YM2149, U6 74LS02, U7 YM2149

Commit message: プリントパターン等検討、ガーバー出力
Parts:
- added J3: IO_CON, Connector_PinHeader_2.54mm:PinHeader_2x07_P2.54mm_Vertical, symbol Connector_Generic:Conn_02x07_Odd_Even
- C1, C2, C3, C6, C7, C8: footprint (none) -> Capacitor_THT:C_Disc_D3.0mm_W1.6mm_P2.50mm
- C4, C5: footprint (none) -> Capacitor_THT:CP_Radial_D5.0mm_P2.50mm
- J1: footprint (none) -> AJ-1780:AJ-1780-2
- J2: footprint (none) -> Connector_PinHeader_2.54mm:PinHeader_2x25_P2.54mm_Horizontal
- JP1, JP2: footprint (none) -> Connector_PinHeader_2.54mm:PinHeader_1x03_P2.54mm_Vertical
- R1, R2, R3, R4: footprint (none) -> Resistor_THT:R_Axial_DIN0207_L6.3mm_D2.5mm_P10.16mm_Horizontal
- U1, U2, U6: footprint (none) -> Package_DIP:DIP-14_W7.62mm_Socket
Connections:
- net GND: now also J3.14 (Pin_14)
- net VCC: now also J3.13 (Pin_13)
- net PA7: now reaches U4.14 (IOA7)
- net PA7: now also J3.8 (Pin_8)
- net PA6: now reaches U4.15 (IOA6)
- net PA6: now also J3.7 (Pin_7)
- net PA5: now reaches U4.16 (IOA5)
- net PA5: now also J3.6 (Pin_6)
- net PA4: now reaches U4.17 (IOA4)
- net PA4: now also J3.5 (Pin_5)
- net PA3: now reaches U4.18 (IOA3)
- net PA3: now also J3.4 (Pin_4)
- net PA2: now reaches U4.19 (IOA2)
- net PA2: now also J3.3 (Pin_3)
- net PA1: now reaches U4.20 (IOA1)
- net PA1: now also J3.2 (Pin_2)
- net PA0: now reaches U4.21 (IOA0)
- net PA0: now also J3.1 (Pin_1)
- no-connect marks 75 -> 71
